Commit message: chore: rename package from hospital_sim to hospital-agv-sim

File: urdf/sensors/imu.xacro (robot description, xacro)
@@ -5,5 +5,5 @@
       <visual>
           <geometry>
-              <mesh filename="package://hospital_sim/meshes/imu_Link.STL" />
+              <mesh filename="package://hospital-agv-sim/meshes/imu_Link.STL" />
           </geometry>
           <material name="red"/>

File: urdf/sensors/lidar.xacro (robot description, xacro)
@@ -6,5 +6,5 @@
         <origin xyz="0 0 0" rpy="1.5708 0 0"/>
         <geometry>
-          <mesh filename="package://hospital_sim/meshes/lidar_Link.STL" />
+          <mesh filename="package://hospital-agv-sim/meshes/lidar_Link.STL" />
         </geometry>
         <material name="green"/>
@@ -13,5 +13,5 @@
         <origin xyz="0 0 0" rpy="1.5708 0 0"/>
         <geometry>
-          <mesh filename="package://hospital_sim/meshes/lidar_Link.STL" />
+          <mesh filename="package://hospital-agv-sim/meshes/lidar_Link.STL" />
         </geometry>
       </collision>

File: urdf/sensors/odom.xacro (robot description, xacro)
@@ -11,5 +11,5 @@
         <origin xyz="0 0 0" rpy="0 0 0"/>
         <geometry>
-           <mesh filename="package://hospital_sim/meshes/rueda_izquierda_Link.STL" />
+           <mesh filename="package://hospital-agv-sim/meshes/rueda_izquierda_Link.STL" />
         </geometry>
         <material name="black"/>
@@ -37,5 +37,5 @@
         <origin xyz="0 0 0" rpy="0 0 0"/>
         <geometry>
-           <mesh filename="package://hospital_sim/meshes/rueda_derecha_Link.STL" />
+           <mesh filename="package://hospital-agv-sim/meshes/rueda_derecha_Link.STL" />
         </geometry>
         <material name="black"/>

File: urdf/tracer2.xacro (robot description, xacro)
@@ -1,12 +1,12 @@
 <?xml version="1.0" encoding="utf-8"?>
 <robot name="tracer2" xmlns:xacro="http://www.ros.org/wiki/xacro">
-  <xacro:include filename="$(find hospital_sim)/urdf/materials.xacro" />
-  <xacro:include filename="$(find hospital_sim)/urdf/tracer2.gazebo" />
-  <xacro:include filename="$(find hospital_sim)/urdf/sensors/odom.xacro" />
-  <xacro:include filename="$(find hospital_sim)/urdf/sensors/imu.xacro" />
-  <xacro:include filename="$(find hospital_sim)/urdf/sensors/lidar.xacro" />
-  <xacro:include filename="$(find hospital_sim)/urdf/sensors/camera.xacro" />
-  <xacro:include filename="$(find hospital_sim)/urdf/sensors/livox_mid70.xacro" />
-  <xacro:include filename="$(find hospital_sim)/urdf/sensors/livox_mid360.xacro"/>
+  <xacro:include filename="$(find hospital-agv-sim)/urdf/materials.xacro" />
+  <xacro:include filename="$(find hospital-agv-sim)/urdf/tracer2.gazebo" />
+  <xacro:include filename="$(find hospital-agv-sim)/urdf/sensors/odom.xacro" />
+  <xacro:include filename="$(find hospital-agv-sim)/urdf/sensors/imu.xacro" />
+  <xacro:include filename="$(find hospital-agv-sim)/urdf/sensors/lidar.xacro" />
+  <xacro:include filename="$(find hospital-agv-sim)/urdf/sensors/camera.xacro" />
+  <xacro:include filename="$(find hospital-agv-sim)/urdf/sensors/livox_mid70.xacro" />
+  <xacro:include filename="$(find hospital-agv-sim)/urdf/sensors/livox_mid360.xacro"/>
   <link name="base_footprint"/>
   <joint name="base_joint" type="fixed">
@@ -24,5 +24,5 @@
       <origin xyz="0 0 0" rpy="0 0 0" />
       <geometry>
-        <mesh filename="package://hospital_sim/meshes/base_link.STL" />
+        <mesh filename="package://hospital-agv-sim/meshes/base_link.STL" />
       </geometry>
       <material name="orange"/>
@@ -43,5 +43,5 @@
         <origin xyz="0 0 0" rpy="0 0 0"/>
         <geometry>
-           <mesh filename="package://hospital_sim/meshes/${name}.STL" />
+           <mesh filename="package://hospital-agv-sim/meshes/${name}.STL" />
         </geometry>
         <material name="green"/>
